File: PCB/YamhillJFETPreamp/YamhillJFETPreamp.kicad_sch (KiCad schematic)
At the start: 25 parts, among them J1 +12 VDC, J2 Output, J3 Input (50 Ω), Q1 2N4401, Q2 2N4401

Commit message: Update arch document
Parts:
- removed C1, C2: 100u, Capacitor_THT:CP_Radial_D6.3mm_P2.50mm, symbol Device:C_Polarized_US
- removed C3: 22u, Capacitor_THT:CP_Radial_D5.0mm_P2.00mm, symbol Device:C_Polarized_US
- removed C4: 100u, Capacitor_THT:CP_Radial_D8.0mm_P3.50mm, symbol Device:C_Polarized_US
- removed C5: 100n, Capacitor_THT:C_Rect_L7.0mm_W2.5mm_P5.00mm, symbol Device:C_Small
- removed C6: 1u, Capacitor_THT:CP_Radial_D6.3mm_P2.50mm, symbol Device:C_Polarized_US
- removed J2: Output, Connector_PinHeader_2.54mm:PinHeader_1x02_P2.54mm_Vertical, symbol Connector_Generic:Conn_01x02
- removed J3: Input (50 Ω), Connector_PinHeader_2.54mm:PinHeader_1x02_P2.54mm_Vertical, symbol Connector_Generic:Conn_01x02
- removed L1: 250u, EtherkitKicadLibrary:T37-V, symbol Device:L
- removed Q1, Q2: 2N4401, Package_TO_SOT_THT:TO-92, symbol EtherkitKicadLibrary:NPN
- removed R7, R9: 1.8k, Resistor_THT:R_Axial_DIN0207_L6.3mm_D2.5mm_P2.54mm_Vertical, symbol Device:R_US
- removed R8: 22, Resistor_THT:R_Axial_DIN0207_L6.3mm_D2.5mm_P2.54mm_Vertical, symbol Device:R_US
- added C1, C2: 100n, symbol Device:C_Small
- added J2, J3: SMA, symbol EtherkitKicadLibrary:BNC
- added J4: MUTE, symbol Connector_Generic:Conn_01x02
- added L1: FB2402-43 3T, symbol Device:L_Iron
- added Q1: J310, symbol Simulation_SPICE:NJFET
- added Q2, Q3: 2N7000, symbol Simulation_SPICE:NMOS
- added T1: FT37-43 15T:5T, symbol EtherkitKicadLibrary:TRANSFORMER_STEP
- J1: value +12 VDC -> +12VDC; footprint Connector_PinHeader_2.54mm:PinHeader_1x02_P2.54mm_Vertical -> (none)
- R1: value 51 -> 100; footprint Resistor_THT:R_Axial_DIN0207_L6.3mm_D2.5mm_P2.54mm_Vertical -> (none)
- R2: value 150 -> 680; footprint Resistor_THT:R_Axial_DIN0207_L6.3mm_D2.5mm_P2.54mm_Vertical -> (none)
- R3: value 680 -> 120; footprint Resistor_THT:R_Axial_DIN0207_L6.3mm_D2.5mm_P2.54mm_Vertical -> (none)
- R4: value 910 -> 120; footprint Resistor_THT:R_Axial_DIN0207_L6.3mm_D2.5mm_P2.54mm_Vertical -> (none)
- R5: value 270 -> 10k; footprint Resistor_THT:R_Axial_DIN0207_L6.3mm_D2.5mm_P2.54mm_Vertical -> (none)
- R6: value 51 -> 10k; footprint Resistor_THT:R_Axial_DIN0207_L6.3mm_D2.5mm_P2.54mm_Vertical -> (none)
- renumbered H2 to H1, H1 to H2, H4 to H3, H3 to H4
Connections:
- net GND: now also R6.2, C1.2, J2.2 (Ext), J3.2 (Ext), J4.1 (Pin_1), Q1.2 (G), Q2.3 (S), Q3.3 (S), T1.4; no longer R5.2
- net at R1.2: now also Q1.1 (D); no longer R3.1
- net at R2.2: now also R1.1, T1.2; no longer R4.1
- net at R4.2: now also Q2.1 (D)
- net +12V: now reaches R5.1
- net +12V: now also J1.1 (Pin_1), R3.1
- net at R3.2: now also R2.1, C1.1, T1.1
- net at R6.1: now also J4.2 (Pin_2), Q3.2 (G)
- new net: C2.1, J3.1 (In)
- new net: C2.2, L1.1, Q1.3 (S)
- new net: J2.1 (In), T1.3
- new net: Q2.2 (G), Q3.1 (D), R5.2
- new net: L1.2, R4.1
Other:
- title: Project Yamhill Audio Feedback Amp -> Project Yamhill
