File: PCB/YamhillAFFeedbackAmp/YamhillAFFeedbackAmp.kicad_pcb (KiCad board)
At the start: 2 copper layers, 50 x 50 mm, 26 parts, among them J1 +12 VDC, J2 Output, J3 Input (50 Ω), Q1 2N4401, Q2 2N4401

Commit message: Update all PCBs for first tranche order
Parts:
- J3: value Input (50 Ω) -> Input
Other:
- board text added: "(50 Ω)"
- board text added: "AF Feedback Amplifier Etherkit 2024"
- board text removed: "AF Feedback Amplifier Etherkit 2023"
Changed lines of the file:
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@@
       (plot_on_all_layers_selection 0x0000000_00000000)
       (disableapertmacros false)
-      (usegerberextensions false)
+      (usegerberextensions true)
       (usegerberattributes true)
       (usegerberadvancedattributes true)
@@
       (plotinvisibletext false)
       (sketchpadsonfab false)
-      (subtractmaskfromsilk false)
+      (subtractmaskfromsilk true)
       (outputformat 1)
       (mirror false)
-      (drillshape 1)
+      (drillshape 0)
       (scaleselection 1)
-      (outputdirectory "")
+      (outputdirectory "fab/")
     )
   )
@@
         (effects (font (size 1 1) (thickness 0.15)))
     )
-    (fp_text value "Input (50 Ω)" (at 0 4.87) (layer "F.SilkS")
+    (fp_text value "Input" (at 0 4.87) (layer "F.SilkS")
         (effects (font (size 1 1) (thickness 0.15)))
     )
@@
     (effects (font (size 1.2 1) (thickness 0.25) bold) (justify left bottom))
   )
+  (gr_text "(50 Ω)" (at 102.6 81) (layer "F.SilkS")
+    (effects (font (size 1 1) (thickness 0.15)) (justify left bottom))
+  )
   (gr_text "Project Yamhill\nCreative Commons CC-BY-SA 4.0" (at 109 97.7) (layer "F.SilkS")
     (effects (font (size 0.9 0.7) (thickness 0.175) bold) (justify left bottom))
   )
-  (gr_text "AF Feedback Amplifier\nEtherkit 2023" (at 109.3 54.9) (layer "F.SilkS")
+  (gr_text "AF Feedback Amplifier\nEtherkit 2024" (at 109.3 54.9) (layer "F.SilkS")
     (effects (font (size 0.9 0.7) (thickness 0.175) bold) (justify left bottom))
   )
