File: PCB/YamhillDiodeRingMixer/YamhillDiodeRingMixer.kicad_pcb (KiCad board)
At the start: 2 copper layers, 50 x 50 mm, 16 parts, among them J1 LO, J2 RF, J3 IF, J4 IF, T1 BN-43-2402 4T Trifilar, T2 BN-43-2402 4T Trifilar

Commit message: Update all PCBs for first tranche order
Parts:
- T1, T2: value BN-43-2402 4T Trifilar -> FT37-43 10T Trifilar; footprint EtherkitKicadLibrary:BN2402_TRIFILAR -> EtherkitKicadLibrary:T37-V-TRIFILARXFMR
- moved T2 8.11 mm to (132.0, 86.0), turned to -90 degrees
- moved T1 6.25 mm to (108.0, 86.0), turned to -90 degrees
Routing:
- net Net-(J2-In): track 6.26 -> 16.3 mm
- net Net-(D1-Pad2): track 17.8 -> 27.7 mm
- net Net-(D3-Pad1): track 28.3 -> 20.6 mm
- net Net-(D1-Pad1): track 17.8 -> 23.1 mm
- net Net-(J1-In): track 13.0 -> 10.8 mm
- net Net-(J3-In): track 25.2 -> 23.2 mm
- net Net-(D2-Pad1): track 19.9 -> 21.4 mm
Other:
- board text added: "Double-Balanced Diode Ring Mixer Etherkit 2024"
- board text removed: "Double-Balanced Diode Ring Mixer Etherkit 2023"
