File: PCB/YamhillDiodeRingMixer/YamhillDiodeRingMixer.kicad_sch (KiCad schematic)
At the start: 14 parts, among them J1 LO, J2 RF, J3 IF, J4 IF, T1 BN-43-2402 4T Trifilar, T2 BN-43-2402 4T Trifilar

Commit message: Update all PCBs for first tranche order
Parts:
- T1, T2: value BN-43-2402 4T Trifilar -> FT37-43 10T Trifilar; footprint EtherkitKicadLibrary:BN2402_TRIFILAR -> EtherkitKicadLibrary:T37-V-TRIFILARXFMR
Changed lines of the file:
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@@
       (effects (font (size 1.27 1.27)))
     )
-    (property "Value" "BN-43-2402 4T Trifilar" (at 109.855 68.453 0)
+    (property "Value" "FT37-43 10T Trifilar" (at 109.855 68.453 0)
       (effects (font (size 1.27 1.27)))
     )
-    (property "Footprint" "EtherkitKicadLibrary:BN2402_TRIFILAR" (at 107.823 81.915 0)
+    (property "Footprint" "EtherkitKicadLibrary:T37-V-TRIFILARXFMR" (at 107.823 81.915 0)
       (effects (font (size 1.524 1.524)) hide)
     )
@@
       (effects (font (size 1.27 1.27)))
     )
-    (property "Value" "BN-43-2402 4T Trifilar" (at 146.558 68.199 0)
+    (property "Value" "FT37-43 10T Trifilar" (at 146.558 68.199 0)
       (effects (font (size 1.27 1.27)))
     )
-    (property "Footprint" "EtherkitKicadLibrary:BN2402_TRIFILAR" (at 148.59 81.788 0)
+    (property "Footprint" "EtherkitKicadLibrary:T37-V-TRIFILARXFMR" (at 148.59 81.788 0)
       (effects (font (size 1.524 1.524)) hide)
     )
