File: PCB/YamhillProtoBoard1x1/YamhillProtoBoard1x1.kicad_pcb (KiCad board)
At the start: 2 copper layers, 50 x 50 mm, 84 parts, among them J1 SMA, J10 Conn_01x02, J11 Conn_01x01, J2 Conn_01x01, J3 Conn_01x02, J4 SMA, J5 Conn_01x02, J6 Conn_01x01

Commit message: Update all PCBs for first tranche order
Other:
- board text added: "Proto Board 1x1 Etherkit 2024"
- board text removed: "Proto Board 1x1 Etherkit 2023"
Changed lines of the file:
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@@
       (plot_on_all_layers_selection 0x0000000_00000000)
       (disableapertmacros false)
-      (usegerberextensions false)
+      (usegerberextensions true)
       (usegerberattributes true)
       (usegerberadvancedattributes true)
@@
       (plotinvisibletext false)
       (sketchpadsonfab false)
-      (subtractmaskfromsilk false)
+      (subtractmaskfromsilk true)
       (outputformat 1)
       (mirror false)
-      (drillshape 1)
+      (drillshape 0)
       (scaleselection 1)
-      (outputdirectory "")
+      (outputdirectory "fab/")
     )
   )
@@
     (effects (font (size 0.9 0.7) (thickness 0.175) bold) (justify left bottom mirror))
   )
-  (gr_text "Proto Board 1x1\nEtherkit 2023" (at 141.1 60.9) (layer "B.SilkS")
+  (gr_text "Proto Board 1x1\nEtherkit 2024" (at 141.1 60.9) (layer "B.SilkS")
     (effects (font (size 0.9 0.7) (thickness 0.175) bold) (justify left bottom mirror))
   )
