File: PCB/YamhillDualDoubleTunedCircuit/YamhillDualDoubleTunedCircuit.kicad_pcb (KiCad board)
At the start: 2 copper layers, 50 x 50 mm, 28 parts, among them J1 SMA, J2 Filter Sel, J3 Filter Sel, J4 SMA

Commit message: Update all PCBs for first tranche order
Other:
- board text added: "Dual Double-Tuned Circuit Etherkit 2024"
- board text removed: "Dual Double-Tuned Circuit Etherkit 2023"
Changed lines of the file:
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@@
       (plot_on_all_layers_selection 0x0000000_00000000)
       (disableapertmacros false)
-      (usegerberextensions false)
+      (usegerberextensions true)
       (usegerberattributes true)
       (usegerberadvancedattributes true)
@@
       (plotinvisibletext false)
       (sketchpadsonfab false)
-      (subtractmaskfromsilk false)
+      (subtractmaskfromsilk true)
       (outputformat 1)
       (mirror false)
-      (drillshape 1)
+      (drillshape 0)
       (scaleselection 1)
-      (outputdirectory "")
+      (outputdirectory "fab/")
     )
   )
@@
     (effects (font (size 0.9 0.7) (thickness 0.175) bold) (justify left bottom))
   )
-  (gr_text "Dual Double-Tuned Circuit\nEtherkit 2023" (at 109.3 54.9) (layer "F.SilkS")
+  (gr_text "Dual Double-Tuned Circuit\nEtherkit 2024" (at 109.3 54.9) (layer "F.SilkS")
     (effects (font (size 0.9 0.7) (thickness 0.175) bold) (justify left bottom))
   )
